File: stekeeb65/led_matrix.kicad_sch (KiCad schematic)
At the start: 66 parts

Commit message: Interim commit before potentially breaking stuff
Parts:
- added S64: QBLP677R-RGB, random-keyboard-parts:QBLP677R-RGB-square_cutout, symbol Device:LED_BGRA
- renumbered S64 to S65, S65 to S66, S66 to S67
Connections:
- net LED2_Col11: now also S64.4 (A)
- net LED_Row_B4: now also S64.1 (BK)
- net LED_Row_G4: now also S64.2 (GK)
- net LED_Row_R4: now also S64.3 (RK)
Changed lines of the file:
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@@
   (junction (at 92.71 123.19) (diameter 0) (color 0 0 0 0)
   )
+  (junction (at 214.63 104.14) (diameter 0) (color 0 0 0 0)
+  )
   (junction (at 134.62 123.19) (diameter 0) (color 0 0 0 0)
   )
@@
   (junction (at 106.68 68.58) (diameter 0) (color 0 0 0 0)
   )
+  (junction (at 204.47 146.05) (diameter 0) (color 0 0 0 0)
+  )
   (junction (at 218.44 128.27) (diameter 0) (color 0 0 0 0)
   )
@@
   (junction (at 232.41 146.05) (diameter 0) (color 0 0 0 0)
   )
+  (junction (at 204.47 156.21) (diameter 0) (color 0 0 0 0)
+  )
   (junction (at 78.74 128.27) (diameter 0) (color 0 0 0 0)
   )
@@
   (junction (at 78.74 110.49) (diameter 0) (color 0 0 0 0)
   )
+  (junction (at 204.47 151.13) (diameter 0) (color 0 0 0 0)
+  )
   (junction (at 134.62 128.27) (diameter 0) (color 0 0 0 0)
   )
@@
     (stroke (width 0) (type default) (color 0 0 0 0))
   )
-  (wire (pts (xy 190.5 146.05) (xy 218.44 146.05))
+  (wire (pts (xy 190.5 146.05) (xy 204.47 146.05))
     (stroke (width 0) (type default) (color 0 0 0 0))
   )
@@
     (stroke (width 0) (type default) (color 0 0 0 0))
   )
+  (wire (pts (xy 204.47 154.94) (xy 204.47 156.21))
+    (stroke (width 0) (type default) (color 0 0 0 0))
+  )
   (wire (pts (xy 162.56 54.61) (xy 162.56 55.88))
     (stroke (width 0) (type default) (color 0 0 0 0))
@@
     (stroke (width 0) (type default) (color 0 0 0 0))
   )
+  (wire (pts (xy 204.47 151.13) (xy 218.44 151.13))
+    (stroke (width 0) (type default) (color 0 0 0 0))
+  )
   (wire (pts (xy 64.77 123.19) (xy 64.77 121.92))
     (stroke (width 0) (type default) (color 0 0 0 0))
@@
     (stroke (width 0) (type default) (color 0 0 0 0))
   )
-  (wire (pts (xy 190.5 156.21) (xy 218.44 156.21))
+  (wire (pts (xy 190.5 156.21) (xy 204.47 156.21))
     (stroke (width 0) (type default) (color 0 0 0 0))
   )
@@
     (stroke (width 0) (type default) (color 0 0 0 0))
   )
-  (wire (pts (xy 190.5 151.13) (xy 218.44 151.13))
+  (wire (pts (xy 190.5 151.13) (xy 204.47 151.13))
     (stroke (width 0) (type default) (color 0 0 0 0))
   )
@@
     (stroke (width 0) (type default) (color 0 0 0 0))
   )
+  (wire (pts (xy 204.47 144.78) (xy 204.47 146.05))
+    (stroke (width 0) (type default) (color 0 0 0 0))
+  )
   (wire (pts (xy 134.62 55.88) (xy 148.59 55.88))
     (stroke (width 0) (type default) (color 0 0 0 0))
@@
     (stroke (width 0) (type default) (color 0 0 0 0))
   )
+  (wire (pts (xy 204.47 146.05) (xy 218.44 146.05))
+    (stroke (width 0) (type default) (color 0 0 0 0))
+  )
   (wire (pts (xy 134.62 68.58) (xy 134.62 67.31))
     (stroke (width 0) (type default) (color 0 0 0 0))
@@
     (stroke (width 0) (type default) (color 0 0 0 0))
   )
+  (wire (pts (xy 204.47 149.86) (xy 204.47 151.13))
+    (stroke (width 0) (type default) (color 0 0 0 0))
+  )
   (wire (pts (xy 256.54 127) (xy 256.54 149.86))
     (stroke (width 0) (type default) (color 0 0 0 0))
@@
     (stroke (width 0) (type default) (color 0 0 0 0))
   )
+  (wire (pts (xy 214.63 104.14) (xy 214.63 149.86))
+    (stroke (width 0) (type default) (color 0 0 0 0))
+  )
   (wire (pts (xy 78.74 73.66) (xy 92.71 73.66))
     (stroke (width 0) (type default) (color 0 0 0 0))
@@
   )
   (wire (pts (xy 78.74 44.45) (xy 78.74 45.72))
+    (stroke (width 0) (type default) (color 0 0 0 0))
+  )
+  (wire (pts (xy 204.47 156.21) (xy 218.44 156.21))
     (stroke (width 0) (type default) (color 0 0 0 0))
   )
@@
   (symbol (lib_id "Device:LED_BGRA") (at 237.49 149.86 0) (unit 1)
     (in_bom yes) (on_board yes) (fields_autoplaced)
-    (property "Reference" "S65" (id 0) (at 237.49 137.16 0))
+    (property "Reference" "S66" (id 0) (at 237.49 137.16 0))
     (property "Value" "QBLP677R-RGB" (id 1) (at 237.49 139.7 0)
       (effects (font (size 0.762 0.762)))
@@
   (symbol (lib_id "Device:LED_BGRA") (at 251.46 149.86 0) (unit 1)
     (in_bom yes) (on_board yes) (fields_autoplaced)
-    (property "Reference" "S66" (id 0) (at 251.46 137.16 0))
+    (property "Reference" "S67" (id 0) (at 251.46 137.16 0))
     (property "Value" "QBLP677R-RGB" (id 1) (at 251.46 139.7 0)
       (effects (font (size 0.762 0.762)))
@@
     (pin "4")
   )
+  (symbol (lib_id "Device:LED_BGRA") (at 209.55 149.86 0) (unit 1)
+    (in_bom yes) (on_board yes) (fields_autoplaced)
+    (property "Reference" "S64" (id 0) (at 209.55 137.16 0))
+    (property "Value" "QBLP677R-RGB" (id 1) (at 209.55 139.7 0)
+      (effects (font (size 0.762 0.762)))
+    )
+    (property "Footprint" "random-keyboard-parts:QBLP677R-RGB-square_cutout" (id 2) (at 209.55 151.13 0)
+      (effects (font (size 1.27 1.27)) hide)
+    )
+    (property "Datasheet" "~" (id 3) (at 209.55 151.13 0)
+      (effects (font (size 1.27 1.27)) hide)
+    )
+    (pin "1")
+    (pin "2")
+    (pin "3")
+    (pin "4")
+  )
   (symbol (lib_id "Device:LED_BGRA") (at 69.85 72.39 0) (unit 1)
     (in_bom yes) (on_board yes) (fields_autoplaced)
@@
   (symbol (lib_id "Device:LED_BGRA") (at 223.52 149.86 0) (unit 1)
     (in_bom yes) (on_board yes) (fields_autoplaced)
-    (property "Reference" "S64" (id 0) (at 223.52 137.16 0))
+    (property "Reference" "S65" (id 0) (at 223.52 137.16 0))
     (property "Value" "QBLP677R-RGB" (id 1) (at 223.52 139.7 0)
       (effects (font (size 0.762 0.762)))
