File: stekeeb65/stekeeb65.kicad_pcb (KiCad board)
At the start: 2 copper layers, 312.8 x 103.2 mm, 134 parts

Commit message: Committing before changes to PCB
Parts:
- added C1: 0.1u, Capacitor_SMD:C_0805_2012Metric_Pad1.18x1.45mm_HandSolder, F.Cu at (377.1, 246.0)
- added C10: 0.47u, Capacitor_SMD:C_0805_2012Metric_Pad1.18x1.45mm_HandSolder, F.Cu at (130.9, 199.2)
- added C11: 0.1u, Capacitor_SMD:C_0805_2012Metric_Pad1.18x1.45mm_HandSolder, F.Cu at (145.3, 196.2)
- added C12: 0.47u, Capacitor_SMD:C_0805_2012Metric_Pad1.18x1.45mm_HandSolder, F.Cu at (130.9, 205.2)
- added C13: 0.47u, Capacitor_SMD:C_0805_2012Metric_Pad1.18x1.45mm_HandSolder, F.Cu at (145.3, 199.2)
- added C14: 0.47u, Capacitor_SMD:C_0805_2012Metric_Pad1.18x1.45mm_HandSolder, F.Cu at (140.5, 196.2)
- added C15: 0.1u, Capacitor_SMD:C_0805_2012Metric_Pad1.18x1.45mm_HandSolder, F.Cu at (135.7, 196.2)
- added C16: 0.1u, Capacitor_SMD:C_0805_2012Metric_Pad1.18x1.45mm_HandSolder, F.Cu at (130.9, 208.2)
- added C17: 0.47u, Capacitor_SMD:C_0805_2012Metric_Pad1.18x1.45mm_HandSolder, F.Cu at (135.7, 202.2)
- added C18: 0.1u, Capacitor_SMD:C_0805_2012Metric_Pad1.18x1.45mm_HandSolder, F.Cu at (135.7, 205.2)
- added C19: 0.47u, Capacitor_SMD:C_0805_2012Metric_Pad1.18x1.45mm_HandSolder, F.Cu at (135.7, 199.2)
- added C2: 0.1u, Capacitor_SMD:C_0805_2012Metric_Pad1.18x1.45mm_HandSolder, F.Cu at (396.5, 235.9)
- added C20: 0.47u, Capacitor_SMD:C_0805_2012Metric_Pad1.18x1.45mm_HandSolder, F.Cu at (140.5, 199.2)
- added C21: 0.47u, Capacitor_SMD:C_0805_2012Metric_Pad1.18x1.45mm_HandSolder, F.Cu at (150.1, 196.2)
- added C22: 0.1u, Capacitor_SMD:C_0805_2012Metric_Pad1.18x1.45mm_HandSolder, F.Cu at (140.5, 202.2)
- added C23: 0.47u, Capacitor_SMD:C_0805_2012Metric_Pad1.18x1.45mm_HandSolder, F.Cu at (135.7, 208.2)
- added C24: 0.1u, Capacitor_SMD:C_0805_2012Metric_Pad1.18x1.45mm_HandSolder, F.Cu at (130.9, 202.2)
- added C25: 0.47u, Capacitor_SMD:C_0805_2012Metric_Pad1.18x1.45mm_HandSolder, F.Cu at (145.3, 202.2)
- added C26: 0.1u, Capacitor_SMD:C_0805_2012Metric_Pad1.18x1.45mm_HandSolder, F.Cu at (130.9, 196.2)
- added C27: 0.1u, Capacitor_SMD:C_0805_2012Metric_Pad1.18x1.45mm_HandSolder, F.Cu at (140.5, 205.2)
- added C3: 0.1u, Capacitor_SMD:C_0805_2012Metric_Pad1.18x1.45mm_HandSolder, F.Cu at (386.8, 246.0)
- added C4: 0.1u, Capacitor_SMD:C_0805_2012Metric_Pad1.18x1.45mm_HandSolder, F.Cu at (396.9, 231.4)
- added C5: 0.1u, Capacitor_SMD:C_0805_2012Metric_Pad1.18x1.45mm_HandSolder, F.Cu at (391.7, 235.9)
- added C6: 1u, Capacitor_SMD:C_0805_2012Metric_Pad1.18x1.45mm_HandSolder, F.Cu at (391.7, 238.9)
- added C7: 1u, Capacitor_SMD:C_0805_2012Metric_Pad1.18x1.45mm_HandSolder, F.Cu at (401.7, 231.4)
- added C8: 1u, Capacitor_SMD:C_0805_2012Metric_Pad1.18x1.45mm_HandSolder, F.Cu at (381.9, 246.0)
- added C9: 0.1u, Capacitor_SMD:C_0805_2012Metric_Pad1.18x1.45mm_HandSolder, F.Cu at (52.9, 249.9)
- added D100: QBLP677R-RGB, random-keyboard-parts:QBLP677R-RGB, F.Cu at (91.9, 196.1)
- added D101: QBLP677R-RGB, random-keyboard-parts:QBLP677R-RGB, F.Cu at (91.9, 224.2)
- added D102: QBLP677R-RGB, random-keyboard-parts:QBLP677R-RGB, F.Cu at (70.3, 196.1)
- added D103: QBLP677R-RGB, random-keyboard-parts:QBLP677R-RGB, F.Cu at (91.9, 207.3)
- added D104: QBLP677R-RGB, random-keyboard-parts:QBLP677R-RGB, F.Cu at (55.9, 235.4)
- added D105: QBLP677R-RGB, random-keyboard-parts:QBLP677R-RGB, F.Cu at (55.9, 207.3)
- added D106: QBLP677R-RGB, random-keyboard-parts:QBLP677R-RGB, F.Cu at (99.1, 218.5)
- added D107: QBLP677R-RGB, random-keyboard-parts:QBLP677R-RGB, F.Cu at (77.5, 201.7)
- added D108: QBLP677R-RGB, random-keyboard-parts:QBLP677R-RGB, F.Cu at (91.9, 212.9)
- added D109: QBLP677R-RGB, random-keyboard-parts:QBLP677R-RGB, F.Cu at (63.1, 196.1)
- added D110: QBLP677R-RGB, random-keyboard-parts:QBLP677R-RGB, F.Cu at (113.5, 207.3)
- added D111: QBLP677R-RGB, random-keyboard-parts:QBLP677R-RGB, F.Cu at (48.7, 212.9)
- added D112: QBLP677R-RGB, random-keyboard-parts:QBLP677R-RGB, F.Cu at (63.1, 224.2)
- added D113: QBLP677R-RGB, random-keyboard-parts:QBLP677R-RGB, F.Cu at (113.5, 201.7)
- added D114: QBLP677R-RGB, random-keyboard-parts:QBLP677R-RGB, F.Cu at (99.1, 207.3)
- added D115: QBLP677R-RGB, random-keyboard-parts:QBLP677R-RGB, F.Cu at (63.1, 207.3)
- added D116: QBLP677R-RGB, random-keyboard-parts:QBLP677R-RGB, F.Cu at (77.5, 196.1)
- added D117: QBLP677R-RGB, random-keyboard-parts:QBLP677R-RGB, F.Cu at (77.5, 229.8)
- added D118: QBLP677R-RGB, random-keyboard-parts:QBLP677R-RGB, F.Cu at (113.5, 196.1)
- added D119: QBLP677R-RGB, random-keyboard-parts:QBLP677R-RGB, F.Cu at (84.7, 235.4)
- added D120: QBLP677R-RGB, random-keyboard-parts:QBLP677R-RGB, F.Cu at (91.9, 218.5)
- added D121: QBLP677R-RGB, random-keyboard-parts:QBLP677R-RGB, F.Cu at (48.7, 235.4)
- added D122: QBLP677R-RGB, random-keyboard-parts:QBLP677R-RGB, F.Cu at (55.9, 201.7)
- added D123: QBLP677R-RGB, random-keyboard-parts:QBLP677R-RGB, F.Cu at (48.7, 196.1)
- added D124: QBLP677R-RGB, random-keyboard-parts:QBLP677R-RGB, F.Cu at (70.3, 201.7)
- added D125: QBLP677R-RGB, random-keyboard-parts:QBLP677R-RGB, F.Cu at (77.5, 235.4)
- added D126: QBLP677R-RGB, random-keyboard-parts:QBLP677R-RGB, F.Cu at (84.7, 218.5)
- added D127: QBLP677R-RGB, random-keyboard-parts:QBLP677R-RGB, F.Cu at (106.3, 196.1)
- added D128: QBLP677R-RGB, random-keyboard-parts:QBLP677R-RGB, F.Cu at (70.3, 207.3)
- added D129: QBLP677R-RGB, random-keyboard-parts:QBLP677R-RGB, F.Cu at (55.9, 218.5)
- added D130: QBLP677R-RGB, random-keyboard-parts:QBLP677R-RGB, F.Cu at (84.7, 201.7)
- added D131: QBLP677R-RGB, random-keyboard-parts:QBLP677R-RGB, F.Cu at (84.7, 196.1)
- added D132: QBLP677R-RGB, random-keyboard-parts:QBLP677R-RGB, F.Cu at (106.3, 201.7)
- added D133: QBLP677R-RGB, random-keyboard-parts:QBLP677R-RGB, F.Cu at (55.9, 212.9)
- added D134: QBLP677R-RGB, random-keyboard-parts:QBLP677R-RGB, F.Cu at (63.1, 212.9)
- added D68: QBLP677R-RGB, random-keyboard-parts:QBLP677R-RGB, F.Cu at (70.3, 235.4)
- added D69: QBLP677R-RGB, random-keyboard-parts:QBLP677R-RGB, F.Cu at (84.7, 224.2)
- added D70: QBLP677R-RGB, random-keyboard-parts:QBLP677R-RGB, F.Cu at (48.7, 229.8)
- added D71: QBLP677R-RGB, random-keyboard-parts:QBLP677R-RGB, F.Cu at (55.9, 224.2)
- added D72: QBLP677R-RGB, random-keyboard-parts:QBLP677R-RGB, F.Cu at (70.3, 218.5)
- added D73: QBLP677R-RGB, random-keyboard-parts:QBLP677R-RGB, F.Cu at (99.1, 201.7)
- added D74: QBLP677R-RGB, random-keyboard-parts:QBLP677R-RGB, F.Cu at (84.7, 207.3)
- added D75: QBLP677R-RGB, random-keyboard-parts:QBLP677R-RGB, F.Cu at (63.1, 201.7)
- added D76: QBLP677R-RGB, random-keyboard-parts:QBLP677R-RGB, F.Cu at (55.9, 196.1)
- added D77: QBLP677R-RGB, random-keyboard-parts:QBLP677R-RGB, F.Cu at (48.7, 207.3)
- added D78: QBLP677R-RGB, random-keyboard-parts:QBLP677R-RGB, F.Cu at (63.1, 218.5)
- added D79: QBLP677R-RGB, random-keyboard-parts:QBLP677R-RGB, F.Cu at (48.7, 218.5)
- added D80: QBLP677R-RGB, random-keyboard-parts:QBLP677R-RGB, F.Cu at (48.7, 224.2)
- added D81: QBLP677R-RGB, random-keyboard-parts:QBLP677R-RGB, F.Cu at (70.3, 224.2)
- added D82: QBLP677R-RGB, random-keyboard-parts:QBLP677R-RGB, F.Cu at (48.7, 201.7)
- added D83: QBLP677R-RGB, random-keyboard-parts:QBLP677R-RGB, F.Cu at (84.7, 229.8)
- added D84: QBLP677R-RGB, random-keyboard-parts:QBLP677R-RGB, F.Cu at (77.5, 207.3)
- added D85: QBLP677R-RGB, random-keyboard-parts:QBLP677R-RGB, F.Cu at (120.7, 196.1)
- added D86: QBLP677R-RGB, random-keyboard-parts:QBLP677R-RGB, F.Cu at (55.9, 229.8)
- added D87: QBLP677R-RGB, random-keyboard-parts:QBLP677R-RGB, F.Cu at (99.1, 196.1)
- added D88: QBLP677R-RGB, random-keyboard-parts:QBLP677R-RGB, F.Cu at (91.9, 201.7)
- added D89: QBLP677R-RGB, random-keyboard-parts:QBLP677R-RGB, F.Cu at (63.1, 235.4)
- added D90: QBLP677R-RGB, random-keyboard-parts:QBLP677R-RGB, F.Cu at (77.5, 218.5)
- added D91: QBLP677R-RGB, random-keyboard-parts:QBLP677R-RGB, F.Cu at (77.5, 212.9)
- added D92: QBLP677R-RGB, random-keyboard-parts:QBLP677R-RGB, F.Cu at (99.1, 212.9)
- added D93: QBLP677R-RGB, random-keyboard-parts:QBLP677R-RGB, F.Cu at (77.5, 224.2)
- added D94: QBLP677R-RGB, random-keyboard-parts:QBLP677R-RGB, F.Cu at (70.3, 212.9)
- added D95: QBLP677R-RGB, random-keyboard-parts:QBLP677R-RGB, F.Cu at (70.3, 229.8)
- added D96: QBLP677R-RGB, random-keyboard-parts:QBLP677R-RGB, F.Cu at (106.3, 207.3)
- added D97: QBLP677R-RGB, random-keyboard-parts:QBLP677R-RGB, F.Cu at (106.3, 212.9)
- added D98: QBLP677R-RGB, random-keyboard-parts:QBLP677R-RGB, F.Cu at (63.1, 229.8)
- added D99: QBLP677R-RGB, random-keyboard-parts:QBLP677R-RGB, F.Cu at (84.7, 212.9)
- added F1: Polyfuse, Fuse:Fuse_0805_2012Metric_Pad1.15x1.40mm_HandSolder, F.Cu at (57.7, 249.8)
- added IC1: ATMEGA32U4-AU, SamacSys_Parts:QFP80P1200X1200X120-44N, F.Cu at (382.0, 237.2)
- added IC2: IS31FL3733B-TQLS4, SamacSys_Parts:QFP50P900X900X120-49N, F.Cu at (346.9, 235.9)
- added IC3: IS31FL3733B-TQLS4, SamacSys_Parts:QFP50P900X900X120-49N, F.Cu at (335.4, 235.9)
- added J1: TYPE-C-31-M12_13_EDITED, Type-C:HRO-TYPE-C-31-M-12-HandSoldering, F.Cu at (231.5, 200.1)
- added J2: Conn_02x03_Odd_Even, Connector_PinHeader_2.54mm:PinHeader_2x03_P2.54mm_Vertical, F.Cu at (45.6, 246.2)
- added R1: 22, Resistor_SMD:R_0805_2012Metric_Pad1.20x1.40mm_HandSolder, F.Cu at (396.5, 238.9)
- added R10: 20k, Resistor_SMD:R_0805_2012Metric_Pad1.20x1.40mm_HandSolder, F.Cu at (154.8, 199.2)
- added R11: 100k, Resistor_SMD:R_0805_2012Metric_Pad1.20x1.40mm_HandSolder, F.Cu at (145.3, 208.2)
- added R12: 100k, Resistor_SMD:R_0805_2012Metric_Pad1.20x1.40mm_HandSolder, F.Cu at (140.4, 208.2)
- added R13: 20k, Resistor_SMD:R_0805_2012Metric_Pad1.20x1.40mm_HandSolder, F.Cu at (150.1, 202.1)
- added R2: 22, Resistor_SMD:R_0805_2012Metric_Pad1.20x1.40mm_HandSolder, F.Cu at (401.3, 234.4)
- added R3: 10k, Resistor_SMD:R_0805_2012Metric_Pad1.20x1.40mm_HandSolder, F.Cu at (391.6, 241.9)
- added R4: 5.1k, Resistor_SMD:R_0805_2012Metric_Pad1.20x1.40mm_HandSolder, F.Cu at (58.0, 245.4)
- added R5: 5.1k, Resistor_SMD:R_0805_2012Metric_Pad1.20x1.40mm_HandSolder, F.Cu at (52.9, 252.8)
- added R6: 100k, Resistor_SMD:R_0805_2012Metric_Pad1.20x1.40mm_HandSolder, F.Cu at (150.1, 199.2)
- added R7: 100k, Resistor_SMD:R_0805_2012Metric_Pad1.20x1.40mm_HandSolder, F.Cu at (145.3, 205.2)
- added R8: 4.7k, Resistor_SMD:R_0805_2012Metric_Pad1.20x1.40mm_HandSolder, F.Cu at (154.9, 196.2)
- added R9: 4.7k, Resistor_SMD:R_0805_2012Metric_Pad1.20x1.40mm_HandSolder, F.Cu at (150.1, 205.1)
- added SW1: SW_Push, random-keyboard-parts:RS187R05A2DSMTRT, F.Cu at (146.4, 233.1)
- added U1: WE-TVS-82400102, Package_TO_SOT_SMD:SOT-23-6, F.Cu at (53.1, 246.1)
- added Y1: 16MHz, Crystal:Crystal_SMD_3225-4Pin_3.2x2.5mm, F.Cu at (391.9, 232.2)
- D_0, D_1, D_10, D_11, D_12, D_13, D_14, D_15, D_16, D_17, D_18, D_19, D_2, D_20, D_21, D_22, D_23, D_24, D_25, D_26, D_27, D_28, D_29, D_3, D_30, D_31, D_32, D_33, D_34, D_35, D_36, D_37, D_38, D_39, D_4, D_40, D_41, D_42, D_43, D_44, D_45, D_46, D_47, D_48, D_49, D_5, D_50, D_51, D_52, D_53, D_54, D_55, D_56, D_57, D_58, D_59, D_6, D_60, D_61, D_62, D_63, D_64, D_65, D_66, D_7, D_8, D_9: moved to F.Cu
- K_0, K_1, K_10, K_11, K_12, K_14, K_16, K_17, K_18, K_19, K_2, K_20, K_21, K_22, K_23, K_24, K_25, K_26, K_27, K_29, K_3, K_31, K_32, K_33, K_34, K_35, K_36, K_37, K_38, K_39, K_4, K_40, K_41, K_43, K_45, K_46, K_47, K_48, K_49, K_5, K_50, K_51, K_52, K_53, K_54, K_56, K_57, K_6, K_64, K_65, K_66, K_7, K_8, K_9: footprint MX_Alps_Hybrid:MX-1U-NoLED -> MX_Hotswap:MX-Hotswap-1U
- K_13: footprint MX_Alps_Hybrid:MX-2U-NoLED -> MX_Hotswap:MX-Hotswap-2U
- K_15, K_28: footprint MX_Alps_Hybrid:MX-1.5U-NoLED -> MX_Hotswap:MX-Hotswap-1.5U
- K_30, K_55: footprint MX_Alps_Hybrid:MX-1.75U-NoLED -> MX_Hotswap:MX-Hotswap-1.75U
- K_42, K_44: footprint MX_Alps_Hybrid:MX-2.25U-NoLED -> MX_Hotswap:MX-Hotswap-2.25U
- K_58, K_59, K_60, K_62, K_63: footprint MX_Alps_Hybrid:MX-1.25U-NoLED -> MX_Hotswap:MX-Hotswap-1.25U
- K_61: footprint MX_Alps_Hybrid:MX-6.25U-NoLED -> MX_Hotswap:MX-Hotswap-6.25U-ReversedStabilizers
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Connections:
- D_0 pad 1: (no net) -> Row0
- D_0 pad 2: (no net) -> Net-(D_0-Pad2)
- D_1 pad 1: (no net) -> Row0
- D_1 pad 2: (no net) -> Net-(D_1-Pad2)
- D_10 pad 1: (no net) -> Row0
- D_10 pad 2: (no net) -> Net-(D_10-Pad2)
- D_11 pad 1: (no net) -> Row0
- D_11 pad 2: (no net) -> Net-(D_11-Pad2)
- D_12 pad 1: (no net) -> Row0
- D_12 pad 2: (no net) -> Net-(D_12-Pad2)
- D_13 pad 1: (no net) -> Row0
- D_13 pad 2: (no net) -> Net-(D_13-Pad2)
- D_14 pad 1: (no net) -> Row0
- D_14 pad 2: (no net) -> Net-(D_14-Pad2)
- D_15 pad 1: (no net) -> Row1
- D_15 pad 2: (no net) -> Net-(D_15-Pad2)
- D_16 pad 1: (no net) -> Row1
- D_16 pad 2: (no net) -> Net-(D_16-Pad2)
- D_17 pad 1: (no net) -> Row1
- D_17 pad 2: (no net) -> Net-(D_17-Pad2)
- D_18 pad 1: (no net) -> Row1
- D_18 pad 2: (no net) -> Net-(D_18-Pad2)
- D_19 pad 1: (no net) -> Row1
- D_19 pad 2: (no net) -> Net-(D_19-Pad2)
- D_2 pad 1: (no net) -> Row0
- D_2 pad 2: (no net) -> Net-(D_2-Pad2)
- D_20 pad 1: (no net) -> Row1
- D_20 pad 2: (no net) -> Net-(D_20-Pad2)
- D_21 pad 1: (no net) -> Row1
- D_21 pad 2: (no net) -> Net-(D_21-Pad2)
- D_22 pad 1: (no net) -> Row1
- D_22 pad 2: (no net) -> Net-(D_22-Pad2)
- D_23 pad 1: (no net) -> Row1
- D_23 pad 2: (no net) -> Net-(D_23-Pad2)
- D_24 pad 1: (no net) -> Row1
- D_24 pad 2: (no net) -> Net-(D_24-Pad2)
- D_25 pad 1: (no net) -> Row1
- D_25 pad 2: (no net) -> Net-(D_25-Pad2)
- D_26 pad 1: (no net) -> Row1
- D_26 pad 2: (no net) -> Net-(D_26-Pad2)
- D_27 pad 1: (no net) -> Row1
- D_27 pad 2: (no net) -> Net-(D_27-Pad2)
- D_28 pad 1: (no net) -> Row1
- D_28 pad 2: (no net) -> Net-(D_28-Pad2)
- D_29 pad 1: (no net) -> Row1
- D_29 pad 2: (no net) -> Net-(D_29-Pad2)
- D_3 pad 1: (no net) -> Row0
- D_3 pad 2: (no net) -> Net-(D_3-Pad2)
- D_30 pad 1: (no net) -> Row2
- D_30 pad 2: (no net) -> Net-(D_30-Pad2)
- D_31 pad 1: (no net) -> Row2
- D_31 pad 2: (no net) -> Net-(D_31-Pad2)
- D_32 pad 1: (no net) -> Row2
- D_32 pad 2: (no net) -> Net-(D_32-Pad2)
- D_33 pad 1: (no net) -> Row2
- D_33 pad 2: (no net) -> Net-(D_33-Pad2)
- D_34 pad 1: (no net) -> Row2
- D_34 pad 2: (no net) -> Net-(D_34-Pad2)
- D_35 pad 1: (no net) -> Row2
- D_35 pad 2: (no net) -> Net-(D_35-Pad2)
- D_36 pad 1: (no net) -> Row2
- D_36 pad 2: (no net) -> Net-(D_36-Pad2)
- D_37 pad 1: (no net) -> Row2
- D_37 pad 2: (no net) -> Net-(D_37-Pad2)
- D_38 pad 1: (no net) -> Row2
- D_38 pad 2: (no net) -> Net-(D_38-Pad2)
- D_39 pad 1: (no net) -> Row2
- D_39 pad 2: (no net) -> Net-(D_39-Pad2)
- D_4 pad 1: (no net) -> Row0
- D_4 pad 2: (no net) -> Net-(D_4-Pad2)
- D_40 pad 1: (no net) -> Row2
- D_40 pad 2: (no net) -> Net-(D_40-Pad2)
- D_41 pad 1: (no net) -> Row2
- D_41 pad 2: (no net) -> Net-(D_41-Pad2)
- D_42 pad 1: (no net) -> Row2
- D_42 pad 2: (no net) -> Net-(D_42-Pad2)
- D_43 pad 1: (no net) -> Row2
- D_43 pad 2: (no net) -> Net-(D_43-Pad2)
- D_44 pad 1: (no net) -> Row3
- D_44 pad 2: (no net) -> Net-(D_44-Pad2)
- D_45 pad 1: (no net) -> Row3
- D_45 pad 2: (no net) -> Net-(D_45-Pad2)
- D_46 pad 1: (no net) -> Row3
- D_46 pad 2: (no net) -> Net-(D_46-Pad2)
- D_47 pad 1: (no net) -> Row3
- D_47 pad 2: (no net) -> Net-(D_47-Pad2)
- D_48 pad 1: (no net) -> Row3
- D_48 pad 2: (no net) -> Net-(D_48-Pad2)
- D_49 pad 1: (no net) -> Row3
- D_49 pad 2: (no net) -> Net-(D_49-Pad2)
- D_5 pad 1: (no net) -> Row0
- D_5 pad 2: (no net) -> Net-(D_5-Pad2)
- D_50 pad 1: (no net) -> Row3
- D_50 pad 2: (no net) -> Net-(D_50-Pad2)
- D_51 pad 1: (no net) -> Row3
- D_51 pad 2: (no net) -> Net-(D_51-Pad2)
- D_52 pad 1: (no net) -> Row3
- D_52 pad 2: (no net) -> Net-(D_52-Pad2)
- D_53 pad 1: (no net) -> Row3
- D_53 pad 2: (no net) -> Net-(D_53-Pad2)
- D_54 pad 1: (no net) -> Row3
- D_54 pad 2: (no net) -> Net-(D_54-Pad2)
- D_55 pad 1: (no net) -> Row3
- D_55 pad 2: (no net) -> Net-(D_55-Pad2)
- D_56 pad 1: (no net) -> Row3
- D_56 pad 2: (no net) -> Net-(D_56-Pad2)
- D_57 pad 1: (no net) -> Row3
- D_57 pad 2: (no net) -> Net-(D_57-Pad2)
- D_58 pad 1: (no net) -> Row4
- D_58 pad 2: (no net) -> Net-(D_58-Pad2)
- D_59 pad 1: (no net) -> Row4
- D_59 pad 2: (no net) -> Net-(D_59-Pad2)
- D_6 pad 1: (no net) -> Row0
- D_6 pad 2: (no net) -> Net-(D_6-Pad2)
- D_60 pad 1: (no net) -> Row4
- D_60 pad 2: (no net) -> Net-(D_60-Pad2)
- D_61 pad 1: (no net) -> Row4
- D_61 pad 2: (no net) -> Net-(D_61-Pad2)
- D_62 pad 1: (no net) -> Row4
- D_62 pad 2: (no net) -> Net-(D_62-Pad2)
- D_63 pad 1: (no net) -> Row4
- D_63 pad 2: (no net) -> Net-(D_63-Pad2)
- D_64 pad 1: (no net) -> Row4
- D_64 pad 2: (no net) -> Net-(D_64-Pad2)
- D_65 pad 1: (no net) -> Row4
- D_65 pad 2: (no net) -> Net-(D_65-Pad2)
- D_66 pad 1: (no net) -> Row4
- D_66 pad 2: (no net) -> Net-(D_66-Pad2)
- D_7 pad 1: (no net) -> Row0
- D_7 pad 2: (no net) -> Net-(D_7-Pad2)
- D_8 pad 1: (no net) -> Row0
- D_8 pad 2: (no net) -> Net-(D_8-Pad2)
- D_9 pad 1: (no net) -> Row0
- D_9 pad 2: (no net) -> Net-(D_9-Pad2)
- K_0 pad 1: (no net) -> Col0
- K_0 pad 2: (no net) -> Net-(D_0-Pad2)
- K_1 pad 1: (no net) -> Col1
- K_1 pad 2: (no net) -> Net-(D_1-Pad2)
- K_10 pad 1: (no net) -> Col10
- K_10 pad 2: (no net) -> Net-(D_10-Pad2)
- K_11 pad 1: (no net) -> Col11
- K_11 pad 2: (no net) -> Net-(D_11-Pad2)
- K_12 pad 1: (no net) -> Col12
- K_12 pad 2: (no net) -> Net-(D_12-Pad2)
- K_13 pad 1: (no net) -> Col13
- K_13 pad 2: (no net) -> Net-(D_13-Pad2)
- K_14 pad 1: (no net) -> Col14
- K_14 pad 2: (no net) -> Net-(D_14-Pad2)
- K_15 pad 1: (no net) -> Col0
- K_15 pad 2: (no net) -> Net-(D_15-Pad2)
- K_16 pad 1: (no net) -> Col1
- K_16 pad 2: (no net) -> Net-(D_16-Pad2)
- K_17 pad 1: (no net) -> Col2
- K_17 pad 2: (no net) -> Net-(D_17-Pad2)
- K_18 pad 1: (no net) -> Col3
- K_18 pad 2: (no net) -> Net-(D_18-Pad2)
- K_19 pad 1: (no net) -> Col4
- K_19 pad 2: (no net) -> Net-(D_19-Pad2)
- K_2 pad 1: (no net) -> Col2
- K_2 pad 2: (no net) -> Net-(D_2-Pad2)
- K_20 pad 1: (no net) -> Col5
- K_20 pad 2: (no net) -> Net-(D_20-Pad2)
- K_21 pad 1: (no net) -> Col6
- K_21 pad 2: (no net) -> Net-(D_21-Pad2)
- K_22 pad 1: (no net) -> Col7
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Other:
- board size 312.8 x 103.2 mm -> 4.5 x 4.5 mm

Commit message: Adding key layout with leds
Parts:
- removed C27: 0.1u, Capacitor_SMD:C_0805_2012Metric_Pad1.18x1.45mm_HandSolder
- removed D100, D101, D102, D103, D104, D105, D106, D107, D108, D109, D110, D111, D112, D113, D114, D115, D116, D117, D118, D119, D120, D121, D122, D123, D124, D125, D126, D127, D128, D129, D130, D131, D132, D133, D134, D68, D69, D70, D71, D72, D73, D74, D75, D76, D77, D78, D79, D80, D81, D82, D83, D84, D85, D86, D87, D88, D89, D90, D91, D92, D93, D94, D95, D96, D97, D98, D99: QBLP677R-RGB, random-keyboard-parts:QBLP677R-RGB
- removed F1: Polyfuse, Fuse:Fuse_0805_2012Metric_Pad1.15x1.40mm_HandSolder
- removed IC3: IS31FL3733B-TQLS4, SamacSys_Parts:QFP50P900X900X120-49N
- removed J2: Conn_02x03_Odd_Even, Connector_PinHeader_2.54mm:PinHeader_2x03_P2.54mm_Vertical
- removed R13: 20k, Resistor_SMD:R_0805_2012Metric_Pad1.20x1.40mm_HandSolder
- removed SW1: SW_Push, random-keyboard-parts:RS187R05A2DSMTRT
- removed U1: WE-TVS-82400102, Package_TO_SOT_SMD:SOT-23-6
- removed Y1: 16MHz, Crystal:Crystal_SMD_3225-4Pin_3.2x2.5mm
- added C0: 1u, Capacitor_SMD:C_0805_2012Metric_Pad1.18x1.45mm_HandSolder, F.Cu at (164.8, 233.6)
- added F0: Polyfuse, Fuse:Fuse_0805_2012Metric_Pad1.15x1.40mm_HandSolder, F.Cu at (42.7, 239.4)
- added IC0: ATMEGA32U4-AU, SamacSys_Parts:QFP80P1200X1200X120-44N, F.Cu at (145.6, 236.4)
- added J0: Conn_02x03_Odd_Even, Connector_PinHeader_2.54mm:PinHeader_2x03_P2.54mm_Vertical, F.Cu at (35.5, 237.3)
- added R0: 10k, Resistor_SMD:R_0805_2012Metric_Pad1.20x1.40mm_HandSolder, F.Cu at (160.1, 240.0)
- added S0: QBLP677R-RGB, random-keyboard-parts:QBLP677R-RGB, F.Cu at (9.53, 15.0)
- added S1: QBLP677R-RGB, random-keyboard-parts:QBLP677R-RGB, F.Cu at (28.6, 15.0)
- added S10: QBLP677R-RGB, random-keyboard-parts:QBLP677R-RGB, F.Cu at (200.0, 15.0)
- added S11: QBLP677R-RGB, random-keyboard-parts:QBLP677R-RGB, F.Cu at (219.1, 15.0)
- added S12: QBLP677R-RGB, random-keyboard-parts:QBLP677R-RGB, F.Cu at (238.1, 15.0)
- added S13: QBLP677R-RGB, random-keyboard-parts:QBLP677R-RGB, F.Cu at (266.7, 15.0)
- added S14: QBLP677R-RGB, random-keyboard-parts:QBLP677R-RGB, F.Cu at (295.3, 15.0)
- added S15: QBLP677R-RGB, random-keyboard-parts:QBLP677R-RGB, F.Cu at (14.3, 34.1)
- added S16: QBLP677R-RGB, random-keyboard-parts:QBLP677R-RGB, F.Cu at (38.1, 34.1)
- added S17: QBLP677R-RGB, random-keyboard-parts:QBLP677R-RGB, F.Cu at (57.1, 34.1)
- added S18: QBLP677R-RGB, random-keyboard-parts:QBLP677R-RGB, F.Cu at (76.2, 34.1)
- added S19: QBLP677R-RGB, random-keyboard-parts:QBLP677R-RGB, F.Cu at (95.2, 34.1)
- added S2: QBLP677R-RGB, random-keyboard-parts:QBLP677R-RGB, F.Cu at (47.6, 15.0)
- added S20: QBLP677R-RGB, random-keyboard-parts:QBLP677R-RGB, F.Cu at (114.3, 34.1)
- added S21: QBLP677R-RGB, random-keyboard-parts:QBLP677R-RGB, F.Cu at (133.3, 34.1)
- added S22: QBLP677R-RGB, random-keyboard-parts:QBLP677R-RGB, F.Cu at (152.4, 34.1)
- added S23: QBLP677R-RGB, random-keyboard-parts:QBLP677R-RGB, F.Cu at (171.4, 34.1)
- added S24: QBLP677R-RGB, random-keyboard-parts:QBLP677R-RGB, F.Cu at (190.5, 34.1)
- added S25: QBLP677R-RGB, random-keyboard-parts:QBLP677R-RGB, F.Cu at (209.6, 34.1)
- added S26: QBLP677R-RGB, random-keyboard-parts:QBLP677R-RGB, F.Cu at (228.6, 34.1)
- added S27: QBLP677R-RGB, random-keyboard-parts:QBLP677R-RGB, F.Cu at (247.7, 34.1)
- added S28: QBLP677R-RGB, random-keyboard-parts:QBLP677R-RGB, F.Cu at (271.5, 34.1)
- added S29: QBLP677R-RGB, random-keyboard-parts:QBLP677R-RGB, F.Cu at (295.3, 34.1)
- added S3: QBLP677R-RGB, random-keyboard-parts:QBLP677R-RGB, F.Cu at (66.7, 15.0)
- added S30: QBLP677R-RGB, random-keyboard-parts:QBLP677R-RGB, F.Cu at (16.7, 53.1)
- added S31: QBLP677R-RGB, random-keyboard-parts:QBLP677R-RGB, F.Cu at (42.9, 53.1)
- added S32: QBLP677R-RGB, random-keyboard-parts:QBLP677R-RGB, F.Cu at (61.9, 53.1)
- added S33: QBLP677R-RGB, random-keyboard-parts:QBLP677R-RGB, F.Cu at (81.0, 53.1)
- added S34: QBLP677R-RGB, random-keyboard-parts:QBLP677R-RGB, F.Cu at (100.0, 53.1)
- added S35: QBLP677R-RGB, random-keyboard-parts:QBLP677R-RGB, F.Cu at (119.1, 53.1)
- added S36: QBLP677R-RGB, random-keyboard-parts:QBLP677R-RGB, F.Cu at (138.1, 53.1)
- added S37: QBLP677R-RGB, random-keyboard-parts:QBLP677R-RGB, F.Cu at (157.2, 53.1)
- added S38: QBLP677R-RGB, random-keyboard-parts:QBLP677R-RGB, F.Cu at (176.2, 53.1)
- added S39: QBLP677R-RGB, random-keyboard-parts:QBLP677R-RGB, F.Cu at (195.3, 53.1)
- added S4: QBLP677R-RGB, random-keyboard-parts:QBLP677R-RGB, F.Cu at (85.7, 15.0)
- added S40: QBLP677R-RGB, random-keyboard-parts:QBLP677R-RGB, F.Cu at (214.3, 53.1)
- added S41: QBLP677R-RGB, random-keyboard-parts:QBLP677R-RGB, F.Cu at (233.4, 53.1)
- added S42: QBLP677R-RGB, random-keyboard-parts:QBLP677R-RGB, F.Cu at (264.3, 53.1)
- added S43: QBLP677R-RGB, random-keyboard-parts:QBLP677R-RGB, F.Cu at (295.3, 53.1)
- added S44: QBLP677R-RGB, random-keyboard-parts:QBLP677R-RGB, F.Cu at (21.4, 72.2)
- added S45: QBLP677R-RGB, random-keyboard-parts:QBLP677R-RGB, F.Cu at (52.4, 72.2)
- added S46: QBLP677R-RGB, random-keyboard-parts:QBLP677R-RGB, F.Cu at (71.4, 72.2)
- added S47: QBLP677R-RGB, random-keyboard-parts:QBLP677R-RGB, F.Cu at (90.5, 72.2)
- added S48: QBLP677R-RGB, random-keyboard-parts:QBLP677R-RGB, F.Cu at (109.5, 72.2)
- added S49: QBLP677R-RGB, random-keyboard-parts:QBLP677R-RGB, F.Cu at (128.6, 72.2)
- added S5: QBLP677R-RGB, random-keyboard-parts:QBLP677R-RGB, F.Cu at (104.8, 15.0)
- added S50: QBLP677R-RGB, random-keyboard-parts:QBLP677R-RGB, F.Cu at (147.6, 72.2)
- added S51: QBLP677R-RGB, random-keyboard-parts:QBLP677R-RGB, F.Cu at (166.7, 72.2)
- added S52: QBLP677R-RGB, random-keyboard-parts:QBLP677R-RGB, F.Cu at (185.7, 72.2)
- added S53: QBLP677R-RGB, random-keyboard-parts:QBLP677R-RGB, F.Cu at (204.8, 72.2)
- added S54: QBLP677R-RGB, random-keyboard-parts:QBLP677R-RGB, F.Cu at (223.8, 72.2)
- added S55: QBLP677R-RGB, random-keyboard-parts:QBLP677R-RGB, F.Cu at (250.0, 72.2)
- added S56: QBLP677R-RGB, random-keyboard-parts:QBLP677R-RGB, F.Cu at (276.2, 72.2)
- added S57: QBLP677R-RGB, random-keyboard-parts:QBLP677R-RGB, F.Cu at (295.3, 72.2)
- added S58: QBLP677R-RGB, random-keyboard-parts:QBLP677R-RGB, F.Cu at (11.9, 91.2)
- added S59: QBLP677R-RGB, random-keyboard-parts:QBLP677R-RGB, F.Cu at (35.7, 91.2)
- added S6: QBLP677R-RGB, random-keyboard-parts:QBLP677R-RGB, F.Cu at (123.8, 15.0)
- added S60: QBLP677R-RGB, random-keyboard-parts:QBLP677R-RGB, F.Cu at (59.5, 91.2)
- added S61: QBLP677R-RGB, random-keyboard-parts:QBLP677R-RGB, F.Cu at (131.0, 91.2)
- added S62: QBLP677R-RGB, random-keyboard-parts:QBLP677R-RGB, F.Cu at (202.4, 91.2)
- added S63: QBLP677R-RGB, random-keyboard-parts:QBLP677R-RGB, F.Cu at (226.2, 91.2)
- added S64: QBLP677R-RGB, random-keyboard-parts:QBLP677R-RGB, F.Cu at (247.7, 91.2)
- added S65: QBLP677R-RGB, random-keyboard-parts:QBLP677R-RGB, F.Cu at (266.7, 91.2)
- added S66: QBLP677R-RGB, random-keyboard-parts:QBLP677R-RGB, F.Cu at (285.8, 91.2)
- added S7: QBLP677R-RGB, random-keyboard-parts:QBLP677R-RGB, F.Cu at (142.9, 15.0)
- added S8: QBLP677R-RGB, random-keyboard-parts:QBLP677R-RGB, F.Cu at (161.9, 15.0)
- added S9: QBLP677R-RGB, random-keyboard-parts:QBLP677R-RGB, F.Cu at (181.0, 15.0)
- added SW0: SW_Push, random-keyboard-parts:RS187R05A2DSMTRT, F.Cu at (157.7, 232.3)
- added U0: WE-TVS-82400102, Package_TO_SOT_SMD:SOT-23-6, F.Cu at (35.7, 246.9)
- added Y0: 16MHz, Crystal:Crystal_SMD_3225-4Pin_3.2x2.5mm, F.Cu at (140.9, 245.9)
- C1, C2: value 0.1u -> 1u
- C14, C20: value 0.47u -> 0.1u
- C15, C9: value 0.1u -> 0.47u
- C6, C7, C8: value 1u -> 0.1u
- IC1: value ATMEGA32U4-AU -> IS31FL3733B-TQLS4; footprint SamacSys_Parts:QFP80P1200X1200X120-44N -> SamacSys_Parts:QFP50P900X900X120-49N
- R10: value 20k -> 100k
- R11, R12: value 100k -> 20k
- R3: value 10k -> 5.1k
- R5: value 5.1k -> 4.7k
- R6: value 100k -> 4.7k
- R8, R9: value 4.7k -> 100k
- moved C8 357.0 mm to (24.9, 247.1)
- moved R3 349.0 mm to (42.7, 236.4)
- moved R5 328.5 mm to (381.3, 242.9)
- moved C9 314.0 mm to (366.9, 243.0)
- moved C10 265.4 mm to (394.7, 228.5)
- moved C7 256.1 mm to (146.0, 245.2)
- moved C17 255.9 mm to (389.9, 231.5)
- moved C15 252.3 mm to (385.1, 234.5)
- moved C14 251.5 mm to (389.9, 228.5)
- moved R7 250.8 mm to (394.6, 231.4)
- moved C18 250.5 mm to (385.1, 228.5)
- moved R12 247.4 mm to (386.1, 237.5)
- moved R6 247.0 mm to (394.6, 234.4)
- moved C4 246.5 mm to (150.8, 245.2)
- moved R2 245.8 mm to (155.6, 243.0)
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Connections:
- C1 pad 1: +5V -> Net-(C1-Pad1)
- C2 pad 1: +5V -> Net-(C2-Pad1)
- C6 pad 1: Net-(C6-Pad1) -> +5V
- C7 pad 1: Net-(C7-Pad1) -> +5V
- C8 pad 1: Net-(C8-Pad1) -> +5V
- IC1 pad 1: Col9 -> unconnected-(IC1-Pad1)
- IC1 pad 10: MOSI -> unconnected-(IC1-Pad10)
- IC1 pad 11: MISO -> unconnected-(IC1-Pad11)
- IC1 pad 12: Row4 -> GND
- IC1 pad 13: RESET_L -> unconnected-(IC1-Pad13)
- IC1 pad 14: +5V -> unconnected-(IC1-Pad14)
- IC1 pad 15: GND -> unconnected-(IC1-Pad15)
- IC1 pad 16: Net-(C7-Pad1) -> LED1_Col0
- IC1 pad 17: Net-(C8-Pad1) -> LED1_Col1
- IC1 pad 18: MCU_SCL -> LED1_Col2
- IC1 pad 19: MCU_SDA -> LED1_Col3
- IC1 pad 2: +5V -> LED_Row_R0
- IC1 pad 20: Col2 -> +5V
- IC1 pad 21: Col3 -> LED1_Col4
- IC1 pad 22: Col5 -> LED1_Col5
- IC1 pad 23: GND -> LED1_Col6
- IC1 pad 24: +5V -> LED1_Col7
- IC1 pad 25: Col4 -> LED1_Col8
- IC1 pad 26: Col6 -> LED1_Col9
- IC1 pad 27: Col7 -> LED1_Col10
- IC1 pad 28: Row1 -> LED1_Col11
- IC1 pad 29: Row2 -> +5V
- IC1 pad 3: Net-(IC1-Pad3) -> LED_Row_G0
- IC1 pad 30: Row3 -> LED1_Col12
- IC1 pad 31: Col0 -> LED1_Col13
- IC1 pad 32: Col1 -> LED1_Col14
- IC1 pad 33: Col8 -> unconnected-(IC1-Pad33)
- IC1 pad 34: +5V -> GND
- IC1 pad 35: GND -> Net-(IC1-Pad35)
- IC1 pad 37: Col14 -> +5V
- IC1 pad 38: Col13 -> +5V
- IC1 pad 39: Col12 -> +5V
- IC1 pad 4: Net-(IC1-Pad4) -> LED_Row_B0
- IC1 pad 40: Col11 -> Net-(IC1-Pad40)
- IC1 pad 41: Col10 -> MCU_SDA
- IC1 pad 42: unconnected-(IC1-Pad42) -> MCU_SCL
- IC1 pad 44: +5V -> GND
- IC1 pad 6: Net-(C6-Pad1) -> LED_Row_R1
- IC1 pad 7: +5V -> LED_Row_G1
- IC1 pad 8: Row0 -> LED_Row_B1
- IC1 pad 9: SCK -> unconnected-(IC1-Pad9)
- IC2 pad 10: unconnected-(IC2-Pad10) -> LED_Row_G4
- IC2 pad 11: unconnected-(IC2-Pad11) -> LED_Row_B4
- IC2 pad 16: LED1_Col0 -> LED2_Col0
- IC2 pad 17: LED1_Col1 -> LED2_Col1
- IC2 pad 18: LED1_Col2 -> LED2_Col2
- IC2 pad 19: LED1_Col3 -> LED2_Col3
- IC2 pad 2: LED_Row_R0 -> LED_Row_R2
- IC2 pad 21: LED1_Col4 -> LED2_Col4
- IC2 pad 22: LED1_Col5 -> LED2_Col5
- IC2 pad 23: LED1_Col6 -> LED2_Col6
- IC2 pad 24: LED1_Col7 -> LED2_Col7
- IC2 pad 25: LED1_Col8 -> LED2_Col8
- IC2 pad 26: LED1_Col9 -> LED2_Col9
- IC2 pad 27: LED1_Col10 -> LED2_Col10
- IC2 pad 28: LED1_Col11 -> LED2_Col11
- IC2 pad 3: LED_Row_G0 -> LED_Row_G2
- IC2 pad 30: LED1_Col12 -> LED2_Col12
- IC2 pad 31: LED1_Col13 -> LED2_Col13
- IC2 pad 32: LED1_Col14 -> LED2_Col14
- IC2 pad 34: GND -> unconnected-(IC2-Pad34)
- IC2 pad 4: LED_Row_B0 -> LED_Row_B2
- IC2 pad 40: Net-(IC2-Pad40) -> Net-(IC1-Pad40)
- IC2 pad 43: GND -> +5V
- IC2 pad 6: LED_Row_R1 -> LED_Row_R3
- IC2 pad 7: LED_Row_G1 -> LED_Row_G3
- IC2 pad 8: LED_Row_B1 -> LED_Row_B3
- IC2 pad 9: unconnected-(IC2-Pad9) -> LED_Row_R4
- R1 pad 2: Net-(IC1-Pad3) -> Net-(IC0-Pad3)
- R10 pad 1: Net-(IC2-Pad35) -> GND
- R10 pad 2: GND -> Net-(IC2-Pad47)
- R11 pad 1: GND -> Net-(IC1-Pad35)
- R11 pad 2: Net-(IC3-Pad47) -> GND
- R12 pad 1: GND -> Net-(IC2-Pad35)
- R12 pad 2: SHUTDOWN_JP -> GND
- R2 pad 1: Net-(IC1-Pad4) -> Net-(IC0-Pad4)
- R3 pad 1: RESET_L -> Net-(J1-Pad4)
- R3 pad 2: +5V -> GND
- R4 pad 1: Net-(J1-Pad4) -> Net-(J1-Pad10)
- R5 pad 1: Net-(J1-Pad10) -> +5V
- R5 pad 2: GND -> MCU_SCL
- R6 pad 1: GND -> +5V
- R6 pad 2: Net-(IC2-Pad47) -> MCU_SDA
- R8 pad 1: +5V -> GND
- R8 pad 2: MCU_SCL -> SHUTDOWN_JP
- R9 pad 1: +5V -> GND
- R9 pad 2: MCU_SDA -> Net-(IC1-Pad47)

Commit message: Adding layout for diodes, LEDs, edge cuts
Parts:
- removed S14: QBLP677R-RGB, random-keyboard-parts:QBLP677R-RGB
- added JP0: SolderJumper_3_Open, Jumper:SolderJumper-3_P1.3mm_Open_RoundedPad1.0x1.5mm, F.Cu at (102.0, 229.6)
- D_0, D_1, D_10, D_11, D_12, D_13, D_14, D_15, D_16, D_17, D_18, D_19, D_2, D_20, D_21, D_22, D_23, D_24, D_25, D_26, D_27, D_28, D_29, D_3, D_30, D_31, D_32, D_33, D_34, D_35, D_36, D_37, D_38, D_39, D_4, D_40, D_41, D_42, D_43, D_44, D_45, D_46, D_47, D_48, D_49, D_5, D_50, D_51, D_52, D_53, D_54, D_55, D_56, D_57, D_58, D_59, D_6, D_60, D_61, D_62, D_63, D_64, D_65, D_66, D_7, D_8, D_9: footprint Diode_SMD:D_SOD-123 -> random-keyboard-parts:D_SOD-123-Pretty; moved to B.Cu
- K_14: value KEYSW -> EC11; footprint MX_Hotswap:MX-Hotswap-1U -> mini-general-tweaks:RotaryEncoder_Alps_EC11E-Switch-Vertical-EDIT
- S0, S1, S10, S11, S12, S13, S15, S16, S17, S18, S19, S2, S20, S21, S22, S23, S24, S25, S26, S27, S28, S29, S3, S30, S31, S32, S33, S34, S35, S36, S37, S38, S39, S4, S40, S41, S42, S43, S44, S45, S46, S47, S48, S49, S5, S50, S51, S52, S53, S54, S55, S56, S57, S58, S59, S6, S60, S61, S62, S63, S64, S65, S66, S7, S8, S9: moved to B.Cu
- moved D_1 377.6 mm to (36.6, 9.53), turned to 90 degrees
- moved D_2 359.3 mm to (55.6, 9.53), turned to 90 degrees
- moved D_44 349.4 mm to (29.4, 66.7), turned to 90 degrees
- moved D_17 340.1 mm to (65.2, 28.6), turned to 90 degrees
- moved D_31 335.1 mm to (50.9, 47.6), turned to 90 degrees
- moved D_16 331.1 mm to (46.1, 28.6), turned to 90 degrees
- moved D_15 328.1 mm to (22.3, 28.6), turned to 90 degrees
- moved D_30 313.1 mm to (24.7, 47.6), turned to 90 degrees
- moved D_5 308.9 mm to (112.8, 9.53), turned to 90 degrees
- moved D_59 300.0 mm to (43.7, 85.7), turned to 90 degrees
- moved D_0 295.3 mm to (17.5, 9.53), turned to 90 degrees
- moved D_60 291.5 mm to (67.5, 85.7), turned to 90 degrees
- moved D_32 285.5 mm to (69.9, 47.6), turned to 90 degrees
- moved D_18 285.3 mm to (84.2, 28.6), turned to 90 degrees
- moved D_4 276.7 mm to (93.7, 9.53), turned to 90 degrees
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Connections:
- IC0 pad 36: unconnected-(IC0-Pad36) -> RE_B
- IC0 pad 9: SCK -> Net-(IC0-Pad9)
Other:
- board size 4.5 x 4.5 mm -> 303.2 x 97.6 mm

Commit message: Started layout for keyboard. still need to verify LED driver schematic
Parts:
- added H0: MountingHole_Pad, MountingHole:MountingHole_2.2mm_M2_DIN965_Pad_TopOnly, F.Cu at (223.9, 263.6)
- added H1: MountingHole_Pad, MountingHole:MountingHole_2.2mm_M2_DIN965_Pad_TopOnly, F.Cu at (229.3, 258.3)
- added H2: MountingHole_Pad, MountingHole:MountingHole_2.2mm_M2_DIN965_Pad_TopOnly, F.Cu at (240.0, 258.3)
- added H3: MountingHole_Pad, MountingHole:MountingHole_2.2mm_M2_DIN965_Pad_TopOnly, F.Cu at (229.3, 263.6)
- added H4: MountingHole_Pad, MountingHole:MountingHole_2.2mm_M2_DIN965_Pad_TopOnly, F.Cu at (223.9, 269.0)
- added H5: MountingHole_Pad, MountingHole:MountingHole_2.2mm_M2_DIN965_Pad_TopOnly, F.Cu at (224.0, 257.6)
- added H6: MountingHole_Pad, MountingHole:MountingHole_2.2mm_M2_DIN965_Pad_TopOnly, F.Cu at (234.6, 263.6)
- added H7: MountingHole_Pad, MountingHole:MountingHole_2.2mm_M2_DIN965_Pad_TopOnly, F.Cu at (234.6, 258.3)
- added H8: MountingHole_Pad, MountingHole:MountingHole_2.2mm_M2_DIN965_Pad_TopOnly, F.Cu at (229.3, 269.0)
- C0, C1, C10, C11, C12, C13, C14, C15, C16, C17, C18, C19, C2, C20, C21, C22, C23, C24, C25, C26, C3, C4, C5, C6, C7, C8, C9: footprint Capacitor_SMD:C_0805_2012Metric_Pad1.18x1.45mm_HandSolder -> Capacitor_SMD:C_0603_1608Metric_Pad1.08x0.95mm_HandSolder; moved to B.Cu
- F0, IC0, IC1, IC2, JP0, SW0, U0, Y0: moved to B.Cu
- J1: footprint Type-C:HRO-TYPE-C-31-M-12-HandSoldering -> Type-C:HRO-TYPE-C-31-M-12-Assembly; moved to B.Cu
- R0, R1, R10, R11, R12, R2, R3, R4, R5, R6, R7, R8, R9: footprint Resistor_SMD:R_0805_2012Metric_Pad1.20x1.40mm_HandSolder -> Resistor_SMD:R_0603_1608Metric_Pad0.98x0.95mm_HandSolder; moved to B.Cu
- S0, S1, S10, S11, S12, S13, S15, S16, S17, S18, S19, S2, S20, S21, S22, S23, S24, S25, S26, S27, S28, S29, S3, S30, S31, S32, S33, S34, S35, S36, S37, S38, S39, S4, S40, S41, S42, S43, S44, S45, S46, S47, S48, S49, S5, S50, S51, S52, S53, S54, S55, S56, S57, S58, S59, S6, S60, S61, S62, S63, S64, S65, S66, S7, S8, S9: footprint random-keyboard-parts:QBLP677R-RGB -> random-keyboard-parts:QBLP677R-RGB-square_cutout
- moved R12 221.7 mm to (164.7, 250.3), turned to 180 degrees
- moved R5 214.4 mm to (166.8, 243.8), turned to 180 degrees
- moved R6 212.4 mm to (182.8, 250.2), turned to 180 degrees
- moved R10 212.3 mm to (168.9, 246.9), turned to 180 degrees
- moved R9 212.2 mm to (164.2, 247.1), turned to 180 degrees
- moved R8 206.7 mm to (186.8, 272.7), turned to 180 degrees
- moved C13 206.5 mm to (183.6, 276.4), turned to 180 degrees
- moved R7 206.0 mm to (189.2, 247.0), turned to 180 degrees
- moved C18 202.6 mm to (184.8, 259.0), turned to 180 degrees
- moved C14 201.7 mm to (193.6, 275.1), turned to 180 degrees
- moved C17 201.5 mm to (189.2, 249.5), turned to 180 degrees
- moved R11 199.1 mm to (188.9, 268.1), turned to 180 degrees
- moved C11 192.5 mm to (189.2, 252.0), turned to 180 degrees
- moved C22 192.5 mm to (181.2, 270.5), turned to 180 degrees
- moved C15 192.1 mm to (193.6, 249.5), turned to 180 degrees
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Connections:
- J1 pad 7: unconnected-(J1-Pad7) -> Net-(J1-Pad5)
Routing:
- net Row4: track 0.00 -> 299.8 mm, vias 0 -> 5
- net Row0: track 0.00 -> 299.5 mm, vias 0 -> 2
- net Row1: track 0.00 -> 288.5 mm
- net Row2: track 0.00 -> 284.7 mm
- net Row3: track 0.00 -> 280.0 mm
- net Col0: track 0.00 -> 112.3 mm
- net Col14: track 0.00 -> 19.9 mm
- net Net-(D_0-Pad2): track 0.00 -> 9.55 mm
- net Net-(J1-Pad5): track 0.00 -> 9.07 mm
- net Net-(J1-Pad6): track 0.00 -> 7.96 mm
- net Net-(D_66-Pad2): track 0.00 -> 7.42 mm
- net Net-(F0-Pad1): track 0.00 -> 7.34 mm
- net Net-(D_57-Pad2): track 0.00 -> 7.23 mm
- net Net-(D_43-Pad2): track 0.00 -> 7.22 mm
- net Net-(D_29-Pad2): track 0.00 -> 7.20 mm
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
Commit message: Redoing keyboard layout. Adding flex cuts to PCB
Parts:
- removed C23, C25: 0.47u, Capacitor_SMD:C_0603_1608Metric_Pad1.08x0.95mm_HandSolder
- removed C24, C26: 0.1u, Capacitor_SMD:C_0603_1608Metric_Pad1.08x0.95mm_HandSolder
- removed H4, H5, H6, H7, H8: MountingHole_Pad, MountingHole:MountingHole_2.2mm_M2_DIN965_Pad_TopOnly
- added TP0: TestPoint, TestPoint:TestPoint_Pad_D1.0mm, B.Cu at (188.0, 230.0)
- F0: footprint Fuse:Fuse_0805_2012Metric_Pad1.15x1.40mm_HandSolder -> Fuse:Fuse_0603_1608Metric_Pad1.05x0.95mm_HandSolder
- H0, H1, H2, H3: footprint MountingHole:MountingHole_2.2mm_M2_DIN965_Pad_TopOnly -> MountingHole:MountingHole_2.2mm_M2_DIN965_Pad_TopBottom
- moved H2 260.9 mm to (73.8, 57.2)
- moved H0 260.6 mm to (42.9, 76.2)
- moved H3 241.2 mm to (283.4, 28.6)
- moved R2 226.1 mm to (19.5, 15.9), turned to 90 degrees
- moved R1 225.4 mm to (17.7, 15.9), turned to -90 degrees
- moved H1 201.2 mm to (233.3, 57.2)
- moved R3 161.0 mm to (16.2, 5.50)
- moved R4 160.0 mm to (21.6, 5.40)
- moved D_0 158.0 mm to (4.50, 7.10), turned to 180 degrees
- moved S0 158.0 mm to (9.53, 4.03)
- moved S1 158.0 mm to (28.6, 4.03)
- moved F0 153.6 mm to (23.4, 5.40)
- moved D_1 151.4 mm to (33.0, 7.10), turned to 180 degrees
- moved D_29 150.7 mm to (302.5, 28.6)
- moved D_57 150.7 mm to (302.5, 66.7)
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Connections:
- K_14 pad B: RE_A -> RE_B
- K_62 pad 1: Col8 -> Col10
- K_63 pad 1: Col10 -> Col11
- S62 pad 4: LED2_Col8 -> LED2_Col10
- S63 pad 4: LED2_Col9 -> LED2_Col11
Routing:
- net Row4: track 299.8 -> 0.00 mm, vias 5 -> 0
- net Row0: track 299.5 -> 0.00 mm, vias 2 -> 0
- net Row1: track 288.5 -> 0.00 mm
- net Row2: track 284.7 -> 0.00 mm
- net Row3: track 280.0 -> 0.00 mm
- net Col14: track 19.9 -> 0.00 mm
- net Net-(D_1-Pad2): track 0.00 -> 13.3 mm
- net Net-(J1-Pad5): track 9.07 -> 0.00 mm
- net Net-(J1-Pad6): track 7.96 -> 0.00 mm
- net Net-(D_66-Pad2): track 7.42 -> 0.00 mm
- net Net-(F0-Pad1): track 7.34 -> 0.00 mm
- net Net-(D_57-Pad2): track 7.23 -> 0.00 mm
- net Net-(D_43-Pad2): track 7.22 -> 0.00 mm
- net Net-(D_29-Pad2): track 7.20 -> 0.00 mm
- net Net-(D_65-Pad2): track 4.32 -> 0.00 mm
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Other:
- outline, holes or cut-outs redrawn
- rule pad_to_mask_clearance: 0 -> 0.2

Commit message: Finish routing matrix
Parts:
- moved SW0 189.9 mm to (279.2, 46.9)
- moved R0 157.3 mm to (89.5, 88.8)
- moved J0 157.1 mm to (88.2, 80.8)
- moved JP0 146.6 mm to (119.3, 82.7)
- moved C5 146.5 mm to (105.4, 92.4)
- moved IC0 146.2 mm to (103.2, 84.7)
- moved C0 146.1 mm to (114.2, 81.6)
- moved C6 146.1 mm to (95.2, 90.0)
- moved Y0 146.1 mm to (114.2, 85.0)
- moved C2 146.1 mm to (114.2, 88.3)
- moved C3 146.1 mm to (111.2, 81.2)
- moved R5 146.1 mm to (117.2, 90.3)
- moved R6 146.1 mm to (112.2, 91.3)
- moved C7 146.1 mm to (95.3, 79.8)
- moved C1 145.9 mm to (102.6, 77.0)
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Connections:
- K_45 pad 1: Col2 -> Col1
- K_46 pad 1: Col3 -> Col2
- K_47 pad 1: Col4 -> Col3
- K_48 pad 1: Col5 -> Col4
- K_49 pad 1: Col6 -> Col5
- K_50 pad 1: Col7 -> Col6
- K_51 pad 1: Col8 -> Col7
- K_52 pad 1: Col9 -> Col8
- K_53 pad 1: Col10 -> Col9
- K_54 pad 1: Col11 -> Col10
- K_62 pad 1: Col10 -> Col9
- K_63 pad 1: Col11 -> Col10
- S45 pad 4: LED2_Col2 -> LED2_Col1
- S46 pad 4: LED2_Col3 -> LED2_Col2
- S47 pad 4: LED2_Col4 -> LED2_Col3
- S48 pad 4: LED2_Col5 -> LED2_Col4
- S49 pad 4: LED2_Col6 -> LED2_Col5
- S50 pad 4: LED2_Col7 -> LED2_Col6
- S51 pad 4: LED2_Col8 -> LED2_Col7
- S52 pad 4: LED2_Col9 -> LED2_Col8
- S53 pad 4: LED2_Col10 -> LED2_Col9
- S54 pad 4: LED2_Col11 -> LED2_Col10
- S55 pad 1: LED_Row_B3 -> unconnected-(S55-Pad1)
- S55 pad 2: LED_Row_G3 -> unconnected-(S55-Pad2)
- S55 pad 3: LED_Row_R3 -> unconnected-(S55-Pad3)
- S56 pad 1: LED_Row_B3 -> unconnected-(S56-Pad1)
- S56 pad 2: LED_Row_G3 -> unconnected-(S56-Pad2)
- S56 pad 3: LED_Row_R3 -> unconnected-(S56-Pad3)
- S62 pad 1: LED_Row_B4 -> unconnected-(S62-Pad1)
- S62 pad 2: LED_Row_G4 -> unconnected-(S62-Pad2)
- S62 pad 3: LED_Row_R4 -> unconnected-(S62-Pad3)
- S62 pad 4: LED2_Col10 -> LED2_Col9
- S63 pad 1: LED_Row_B4 -> unconnected-(S63-Pad1)
- S63 pad 2: LED_Row_G4 -> unconnected-(S63-Pad2)
- S63 pad 3: LED_Row_R4 -> unconnected-(S63-Pad3)
- S63 pad 4: LED2_Col11 -> LED2_Col10
Routing:
- net LED_Row_B2: track 0.00 -> 491.2 mm, vias 0 -> 27
- net Row2: track 0.00 -> 463.5 mm, vias 0 -> 2
- net LED_Row_G2: track 0.00 -> 435.3 mm, vias 0 -> 7
- net LED_Row_R2: track 0.00 -> 421.0 mm, vias 0 -> 5
- net LED_Row_R1: track 0.00 -> 399.8 mm, vias 0 -> 10
- net LED_Row_B3: track 0.00 -> 381.0 mm, vias 0 -> 29
- net LED_Row_G1: track 0.00 -> 379.6 mm, vias 0 -> 8
- net LED_Row_B1: track 0.00 -> 369.4 mm, vias 0 -> 27
- net LED_Row_R3: track 0.00 -> 345.2 mm, vias 0 -> 8
- net LED_Row_G3: track 0.00 -> 341.6 mm, vias 0 -> 4
- net Row1: track 0.00 -> 325.7 mm
- net Row0: track 0.00 -> 323.7 mm, vias 0 -> 2
- net Row3: track 0.00 -> 320.0 mm
- net LED_Row_B0: track 0.00 -> 315.3 mm, vias 0 -> 27
- net LED_Row_R4: track 0.00 -> 299.3 mm, vias 0 -> 3
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Other:
- outline, holes or cut-outs redrawn
